File: main-board/main-board.kicad_pcb (KiCad board)
At the start: 2 copper layers, 70 x 45.7 mm, 71 parts, among them J1 ECS00065, J2 ECS00094, P1 ECS00029, P2 ECS00015, P3 ECS00067, P4 ECS00029, P5 ECS00029, P6 ECS00067, P7 ECS00067, P8 ECS00013, Q1 ECS00087, Q2 ECS00073, Q3 ECS00087, U1 ECS00017, U2 ECS00032, U3 ECA00002, U4 ECS00030, U5 ECS00016, X1 ECS00006, X2 ECS00005

Commit message: Added output files, gerbers, dril files, raster images, and updates to PCB design files.
Parts:
- removed U1: ECS00017, ECFootprints:ECTQFP-32
- added U201: ECS00017, ECFootprints:ECTQFP-32, F.Cu at (54.9, 67.6)
- renumbered C2 to C201, C4 to C202, C5 to C203, C6 to C204, C7 to C205, C1 to C206, C8 to C207, C3 to C208, C9 to C209, C10 to C210, C21 to C211, C11 to C212, C12 to C213, C13 to C214, C15 to C301, C16 to C302, C19 to C303, C20 to C304, C22 to C305, C24 to C401, D4 to D201, D2 to D301, J1 to J201, J2 to J202, L1 to L201, LED1 to LED201, LED2 to LED202, NT1 to NT201, P8 to P201, P1 to P202, P2 to P203, P4 to P301, P5 to P302, P3 to P303, P6 to P401, P7 to P402, Q1 to Q301, Q2 to Q302, Q3 to Q401, R1 to R201, R2 to R202, R15 to R203, R24 to R204, R3 to R205, R25 to R206, R4 to R207, R6 to R208, R7 to R209, R5 to R210, R8 to R211, R11 to R301, R10 to R302, R23 to R303, R12 to R304, R16 to R305, R17 to R306, R18 to R307, R21 to R308, R13 to R309, R19 to R310, R20 to R401, R14 to R402, R22 to R403, R26 to R404, U2 to U202, U3 to U203, U5 to U301, U4 to U302, X1 to X201, X2 to X202
Connections:
- net +3V3 renamed VDD
