File: main-board/main-board.kicad_pcb (KiCad board)
At the start: 2 copper layers, 70 x 45.7 mm, 71 parts, among them J201 ECS00065, J202 ECS00094, P201 ECS00013, P202 ECS00029, P203 ECS00015, P301 ECS00029, P302 ECS00029, P303 ECS00067, P401 ECS00067, P402 ECS00067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

Commit message: Commit fabrication files.
Other:
- board text added: "0.20 MM 0.20 MM 0.20 MM 0.81 MM"
- board text added: "0.20 MM 0.25 MM 0.20 MM 0.50 MM 0.30 MM"
- board text added: "B-STAGE"
- board text removed: "10 MILS 10 MILS 7.5 MILS 125 MILS"
- board text removed: "10 MILS 25 MILS 0.2 MM 25 MILS 15 MILS"
- board text removed: "B-STAGE (.013 REF)"
Changed lines of the file:
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@@
   (general
     (thickness 1.6)
-    (drawings 87)
+    (drawings 88)
     (tracks 1086)
     (zones 0)
@@
     (visible_elements 7FFFFFFF)
     (pcbplotparams
-      (layerselection 0x00000_ffffffff)
+      (layerselection 0x00200_7ffffffe)
       (usegerberextensions false)
       (usegerberattributes false)
@@
       (excludeedgelayer false)
       (linewidth 0.100000)
-      (plotframeref false)
+      (plotframeref true)
       (viasonmask false)
       (mode 1)
@@
       (drillshape 0)
       (scaleselection 1)
-      (outputdirectory "assembly"))
+      (outputdirectory "fabrication"))
   )
   (net 0 "")
@@
     )
   )
+  (gr_text B-STAGE (at 67 156.3) (layer Cmts.User)
+    (effects (font (size 1.5 1.5) (thickness 0.15)))
+  )
   (gr_line (start 95 155.3) (end 98 155.3) (layer Cmts.User) (width 0.15))
   (gr_line (start 38 162.3) (end 30 162.3) (layer Cmts.User) (width 0.15))
@@
   (gr_line (start 88 146.3) (end 88 152.3) (layer Cmts.User) (width 0.15))
   (gr_line (start 40 146.3) (end 88 146.3) (layer Cmts.User) (width 0.15))
-  (gr_text "B-STAGE (.013 REF)" (at 67 143.3) (layer Cmts.User)
+  (gr_text B-STAGE (at 67 143.3) (layer Cmts.User)
     (effects (font (size 1.5 1.5) (thickness 0.15)))
   )
@@
     (effects (font (size 1.5 1.5) (thickness 0.2)) (justify left))
   )
-  (gr_text "10 MILS\n10 MILS\n7.5 MILS\n125 MILS" (at 255 139.3) (layer Dwgs.User)
+  (gr_text "0.20 MM\n0.20 MM\n0.20 MM\n0.81 MM" (at 255 139.3) (layer Dwgs.User)
     (effects (font (size 1.5 1.5) (thickness 0.2)) (justify left))
   )
-  (gr_text "10 MILS\n25 MILS\n0.2 MM\n25 MILS\n15 MILS" (at 194 140.3) (layer Dwgs.User)
+  (gr_text "0.20 MM\n0.25 MM\n0.20 MM\n0.50 MM\n0.30 MM" (at 194 140.3) (layer Dwgs.User)
     (effects (font (size 1.5 1.5) (thickness 0.2)) (justify left))
   )

Commit message: Commiting power board output files.
Other:
- board text added: "1.6 MM +/- 0.1 MM"
- board text added: "BOT LAYER"
- board text added: "TOP LAYER"
- board text removed: ".063 +/- .005"
- board text removed: "INT2 LAYER"
- board text removed: "TOP LAYER (VOLTAGE/RTN SIGNAL TRACES)"
Changed lines of the file:
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@@
   (gr_line (start 32 162.3) (end 32 151.3) (layer Cmts.User) (width 0.15))
   (gr_line (start 32 136.3) (end 32 145.3) (layer Cmts.User) (width 0.15))
-  (gr_text ".063\n+/- .005" (at 32 148.3) (layer Cmts.User)
+  (gr_text "1.6 MM\n+/- 0.1 MM" (at 32 148.3) (layer Cmts.User)
     (effects (font (size 1.5 1.5) (thickness 0.15)))
   )
@@
     (effects (font (size 1.5 1.5) (thickness 0.15)) (justify left))
   )
-  (gr_text "TOP LAYER (VOLTAGE/RTN SIGNAL TRACES)" (at 98 144.3) (layer Cmts.User)
+  (gr_text "TOP LAYER" (at 98 144.3) (layer Cmts.User)
     (effects (font (size 1.5 1.5) (thickness 0.15)) (justify left))
   )
-  (gr_text "INT2 LAYER" (at 98 155.3) (layer Cmts.User)
+  (gr_text "BOT LAYER" (at 98 155.3) (layer Cmts.User)
     (effects (font (size 1.5 1.5) (thickness 0.15)) (justify left))
   )
