File: power-board/power-board.kicad_pcb (KiCad board)
At the start: 2 copper layers, 70 x 52 mm, 36 parts, among them J1 ECS00066, J11 ECS00059, J8 ECS00059, J9 ECS00059, P1 ECS00067, P12 ECS00068, P13 ECS00068, P2 ECS00007, P3 ECS00013, P4 ECS00004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

Commit message: Commiting power board output files.
Other:
- rule trace_min: 0 -> 0.2
- rule via_min_drill: 0 -> 0.5
- rule via_min_size: 0 -> 0.5
- board text added: "0.20 MM 0.20 MM 0.20 MM 0.81 MM"
- board text added: "0.20 MM 0.25 MM 0.20 MM 0.50 MM 0.30 MM"
- board text added: "1.6 MM +/- 0.1 MM"
- board text added: "B-STAGE"
- board text added: "BOT LAYER"
- board text added: "TOP LAYER"
- board text removed: ".063 +/- .005"
- board text removed: "10 MILS 10 MILS 7.5 MILS 125 MILS"
- board text removed: "10 MILS 25 MILS 0.2 MM 25 MILS 15 MILS"
- board text removed: "B-STAGE (.013 REF)"
- board text removed: "INT2 LAYER"
- board text removed: "TOP LAYER (VOLTAGE/RTN SIGNAL TRACES)"
